File: circuit/PicoTracer.kicad_sch (KiCad schematic)
At the start: 23 parts, among them J1 Conn_01x04_Socket, J10 Conn_01x02_Socket, J2 Conn_01x04_Socket, J3 Conn_01x02_Socket, J4 Conn_02x20_Top_Bottom, J5 Conn_02x20_Top_Bottom, J6 Conn_01x04_Socket, J7 8P8C, J9 Conn_01x02_Socket, SW1 SW_Push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

Commit message: 配線図完成、回路図スイッチの配線位置変更
Connections:
- net +12V: no longer J10.1 (Pin_1)
- net 3.3V: now also J4.5 (Pin_5)
- net Clock: now also J5.34 (Pin_34)
- net Curve_Sensor: now also J4.7 (Pin_7)
- net Din: now also J5.36 (Pin_36)
- net Dout: now also J5.35 (Pin_35)
- net GND: now also J4.3 (Pin_3), J5.23 (Pin_23)
- net Goal_Sensor: now also J4.10 (Pin_10)
- net Left_Direction: now also J4.15 (Pin_15)
- net Left_Enable: now also J4.12 (Pin_12)
- net Left_Step: now also J4.14 (Pin_14)
- net Right_Direction: now also J5.29 (Pin_29)
- net Right_Enable: now also J5.27 (Pin_27)
- net Right_Step: now also J5.31 (Pin_31)
- net Sel1: now also J5.32 (Pin_32)
- net Sel2: now also J5.37 (Pin_37)
- net at J5.19 (Pin_19), R15.2, SW1.1: now also J5.39 (Pin_39)
- net at J4.39 (Pin_39), J6.1 (Pin_1): now also J4.19 (Pin_19)
- net at J4.40 (Pin_40), J6.2 (Pin_2): now also J4.20 (Pin_20)
- net at J4.22 (Pin_22), J6.3 (Pin_3), J7.2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: now also J4.2 (Pin_2)
- net at J5.20 (Pin_20), R16.2, SW2.2: now also J5.40 (Pin_40)
- net at J4.1 (Pin_1): now also J4.21 (Pin_21)
- net at J4.11 (Pin_11): now also J4.31 (Pin_31), Reset_SW1.1
- net at J4.13 (Pin_13): now also J4.33 (Pin_33), Reset_SW1.2
- net at J4.16 (Pin_16): now also J4.36 (Pin_36)
- net at J4.17 (Pin_17): now also J4.37 (Pin_37)
- net at J4.18 (Pin_18): now also J4.38 (Pin_38)
- net at J4.24 (Pin_24): now also J4.4 (Pin_4)
- net at J4.26 (Pin_26): now also J4.6 (Pin_6)
- net at J4.28 (Pin_28): now also J4.8 (Pin_8)
- net at J4.29 (Pin_29), R1.1, R2.2: now also J4.9 (Pin_9)
- net at Left1.8 (VMOT), R2.1, Right1.8 (VMOT)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: now also J10.1 (Pin_1)
- net at BZ1.1 (+), J5.8 (Pin_8): now also J5.28 (Pin_28)
- net at BZ1.2 (-), J5.6 (Pin_6): now also J5.26 (Pin_26)
- net at J5.1 (Pin_1): now also J5.21 (Pin_21)
- net at J5.10 (Pin_10): now also J5.30 (Pin_30)
- net at J5.13 (Pin_13): now also J5.33 (Pin_33)
- net at J5.18 (Pin_18): now also J5.38 (Pin_38)
- net at J5.2 (Pin_2): now also J5.22 (Pin_22)
- net at J5.24 (Pin_24): now also J5.4 (Pin_4)
- net at J5.25 (Pin_25): now also J5.5 (Pin_5)
- no-connect marks 62 -> 8
