File: circuit/PicoTracer.kicad_pcb (KiCad board)
At the start: 2 copper layers, 105 x 85 mm, 23 parts, among them J1 Conn_01x04_Socket, J10 Conn_01x02_Socket, J2 Conn_01x04_Socket, J3 Conn_01x02_Socket, J4 Conn_02x20_Top_Bottom, J5 Conn_02x20_Top_Bottom, J6 Conn_01x04_Socket, J7 8P8C, J9 Conn_01x02_Socket, SW1 SW_Push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

Commit message: PicoTracer-backupsファイルを管理外に変更　センサー、メイン配線図ファイル修正、その他ファイル更新
Other:
- board text added: "SCL"
- board text added: "SDA"
Changed lines of the file:
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@@
 		(layer "Edge.Cuts")
+	)
+	(gr_text "SCL"
+		(at 142.24 63.5 0)
+		(layer "Edge.Cuts")
+		(effects
+			(font
+				(size 1 1)
+				(thickness 0.15)
+			)
+			(justify left bottom)
+		)
+	)
+	(gr_text "SDA"
+		(at 127 63.5 0)
+		(layer "Edge.Cuts")
+		(effects
+			(font
+				(size 1 1)
+				(thickness 0.15)
+			)
+			(justify left bottom)
+		)
+	)
+	(gr_text "SDA"
+		(at 142.24 60.96 0)
+		(layer "Edge.Cuts")
+		(effects
+			(font
+				(size 1 1)
+				(thickness 0.15)
+			)
+			(justify left bottom)
+		)
+	)
+	(gr_text "SCL"
+		(at 121.92 63.5 0)
+		(layer "Edge.Cuts")
+		(effects
+			(font
+				(size 1 1)
+				(thickness 0.15)
+			)
+			(justify left bottom)
+		)
 	)
 	(segment
